File: tone-selector/tone-selector.kicad_pcb (KiCad board)
At the start: 2 copper layers, 66 x 59.7 mm, 18 parts, among them SW51 switch5pos, U1 LM555N, U2 LM555N

Commit message: Atualizado com a malha
Routing:
- added copper zone on B.Cu, net GND
Changed lines of the file:
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@@
   (segment (start 214.63 139.7) (end 210.82 135.89) (width 0.5) (layer B.Cu) (net 16))
   (segment (start 214.63 142.24) (end 214.63 139.7) (width 0.5) (layer B.Cu) (net 16))
+  (zone (net 2) (net_name GND) (layer B.Cu) (hatch edge 0.508)
+    (connect_pads (clearance 0.508))
+    (min_thickness 0.254)
+    (fill yes (arc_segments 16) (thermal_gap 0.508) (thermal_bridge_width 0.508))
+    (polygon
+      (pts
+        (xy 224.155 153.67) (xy 160.02 153.67) (xy 160.02 95.25) (xy 224.155 95.25) (xy 224.155 153.67)
+      )
+    )
+  )
 )
